File: IP2312_Battery_Charger_PCB/IP2312_Battery_Charger_PCB.kicad_sch (KiCad schematic)
At the start: 0 parts

Commit message: Schematic
Parts:
- added C1: 100nF, symbol Device:C
- added C4, C7, C8: 22uF, symbol Device:C
- added C5, C6: 10uF, symbol Device:C
- added D1: CHG, symbol Device:LED_Filled
- added D2: FULL, symbol Device:LED_Filled
- added J1, J2: Jumper, symbol MyLib:Jumper
- added J10, J3, J4, J5, J6, J7, J8, J9: (no value), symbol MyLib:Jumper
- added L1: 2.2uH, symbol Device:L
- added R1, R2: 5.1k, symbol Device:R
- added R10: 560k, symbol Device:R
- added R11: 510k, symbol Device:R
- added R12: 180k, symbol Device:R
- added R13, R5: 75k, symbol Device:R
- added R17: 1R, symbol Device:R
- added R18: 100k, symbol Device:R
- added R19, R3: 1k, symbol Device:R
- added R20: 51k, symbol Device:R
- added R21: 0.5R, symbol Device:R
- added R4: 43k, symbol Device:R
- added R6, R7: 100R, symbol Device:R
- added R8: 82k, symbol Device:R
- added R9: NTC, symbol Device:R
- added U1: IP2312U_VSET, symbol MyLib:IP2312U_VSET
- added U2: XB5606AJ, symbol MyLib:XB5606AJ
- added USB1: USB_C_Receptacle_PowerOnly_6P, symbol Connector:USB_C_Receptacle_PowerOnly_6P
Connections:
- new net: C7.1, R21.2, U1.5 (BAT)
- new net: R18.1, R4.1, R5.1, R6.1, U1.1 (D1)
- new net: J3., R4.2
- new net: J7., R20.1
- new net: C1.2, J2., U2.3 (VDD)
- new net: R7.1, U1.3 (D2)
- new net: D2.2 (A), R7.2
- new net: R1.1, USB1.A5 (CC1)
- new net: R19.1, U1.2 (TEST)
- new net: J6., R8.1, R9.1
- new net: R10.1, R11.1, R12.1, R13.1, U1.6 (ICHG)
- new net: C5.1, R17.2
- new net: J4., R5.2
- new net: J6., J7., U1.4 (NTC)
- new net: J8., R11.2
- new net: J5., R18.2
- new net: J9., R12.2
- new net: L1.1, U1.7 (SW)
- new net: J2., R3.1
- new net: D1.2 (A), R6.2
- new net: R2.1, USB1.B5 (CC2)
- new net: J10., R13.2
- new net B+: C8.1, L1.2, R19.2, R21.1, R3.2
- new net B-: C1.1, J1., U2.1 (GND), U2.2 (GND)
- new net GND: C4.2, C5.2, C6.2, C7.2, C8.2, D1.1 (K), D2.1 (K), J1., J10., J3., J4., J5., J8., J9., R1.2, R10.2, R2.2, R20.2, R8.2, R9.2, U1.9 (EPAD), U2.4 (VM), U2.5 (VM), USB1.A12 (GND), USB1.B12 (GND), USB1.SH (SHIELD)
- new net VCC: C4.1, C6.1, R17.1, U1.8 (VIN), USB1.A9 (VBUS), USB1.B9 (VBUS)
Other:
- company: (none) -> FETEL-HCMUS
- title: (none) -> Mạch sạc pin Lion

Commit message: Footprint + PCB setup
Parts:
- C1: footprint (none) -> Capacitor_SMD:C_0402_1005Metric
- C2: renamed from C7; footprint (none) -> Capacitor_SMD:C_0805_2012Metric
- C3: renamed from C8; footprint (none) -> Capacitor_SMD:C_0805_2012Metric
- C4, C5, C6: footprint (none) -> Capacitor_SMD:C_0805_2012Metric
- D1, D2: footprint (none) -> LED_SMD:LED_0603_1608Metric
- J1: value Jumper -> J1; footprint (none) -> MyLib_Footprint:Jumper_0603_1608Metric
- J10: value (none) -> S3; footprint (none) -> MyLib_Footprint:Jumper_0603_1608Metric
- J2: value Jumper -> J2; footprint (none) -> MyLib_Footprint:Jumper_0603_1608Metric
- J3: value (none) -> B1; footprint (none) -> MyLib_Footprint:Jumper_0603_1608Metric
- J4: value (none) -> B2; footprint (none) -> MyLib_Footprint:Jumper_0603_1608Metric
- J5: value (none) -> B3; footprint (none) -> MyLib_Footprint:Jumper_0603_1608Metric
- J6: value (none) -> T0; footprint (none) -> MyLib_Footprint:Jumper_0603_1608Metric
- J7: value (none) -> T1; footprint (none) -> MyLib_Footprint:Jumper_0603_1608Metric
- J8: value (none) -> S1; footprint (none) -> MyLib_Footprint:Jumper_0603_1608Metric
- J9: value (none) -> S2; footprint (none) -> MyLib_Footprint:Jumper_0603_1608Metric
- L1: footprint (none) -> Inductor_SMD:L_Sunlord_MWSA0603S
- R1, R2: footprint (none) -> Resistor_SMD:R_0402_1005Metric
- R10: renamed from R6; footprint (none) -> Resistor_SMD:R_0603_1608Metric
- R11: renamed from R7; footprint (none) -> Resistor_SMD:R_0603_1608Metric
- R12: renamed from R20; footprint (none) -> Resistor_SMD:R_0603_1608Metric
- R13: renamed from R8; footprint (none) -> Resistor_SMD:R_0603_1608Metric
- R14: renamed from R4; footprint (none) -> Resistor_SMD:R_0603_1608Metric
- R15: renamed from R5; footprint (none) -> Resistor_SMD:R_0603_1608Metric
- R16: renamed from R18; footprint (none) -> Resistor_SMD:R_0603_1608Metric
- R17, R3: footprint (none) -> Resistor_SMD:R_0603_1608Metric
- R18: renamed from R9; footprint (none) -> Resistor_SMD:R_0603_1608Metric
- R4: renamed from R21; footprint (none) -> Resistor_SMD:R_0603_1608Metric
- R5: renamed from R10; footprint (none) -> Resistor_SMD:R_0603_1608Metric
- R6: renamed from R11; footprint (none) -> Resistor_SMD:R_0603_1608Metric
- R7: renamed from R12; footprint (none) -> Resistor_SMD:R_0603_1608Metric
- R8: renamed from R13; footprint (none) -> Resistor_SMD:R_0603_1608Metric
- R9: renamed from R19; footprint (none) -> Resistor_SMD:R_0603_1608Metric
- U1: footprint (none) -> MyLib_Footprint:HSOP-8-1EP_3.9x4.9mm_P1.27mm_EP2.3x2.3mm_ThermalVias-IP2312
- U2: footprint (none) -> MyLib_Footprint:SOT-23-5-XB5606AJ
- USB1: footprint (none) -> MyLib_Footprint:USB-C_Receptacle_GCT_USB4125-xx-x-0190_6P_TopMnt_Horizontal
Connections:
- net B-: now also J1.2; no longer J1.
- net GND: now also J1.1, J10.2, J3.2, J4.2, J5.2, J8.2, J9.2; no longer J1., J10., J3., J4., J5., J8., J9.
- net at R14.2: now also J3.1; no longer J3.
- net at R12.1: now also J7.2; no longer J7.
- net at C1.2, U2.3 (VDD): now also J2.1; no longer J2.
- net at R13.1, R18.1: now also J6.2; no longer J6.
- net at R15.2: now also J4.1; no longer J4.
- net at R6.2: now also J8.1; no longer J8.
- net at R16.2: now also J5.1; no longer J5.
- net at R7.2: now also J9.1; no longer J9.
- net at R3.1: now also J2.2; no longer J2.
- net at R8.2: now also J10.1; no longer J10.
- new net: J6.1, J7.1, U1.4 (NTC)
