File: IP2312_Battery_Charger_PCB/IP2312_Battery_Charger_PCB.kicad_pcb (KiCad board)
At the start: 2 copper layers, 36 x 18 mm, 40 parts, among them J1 J1, J10 S3, J2 J2, J3 B1, J4 B2, J5 B3, J6 T0, J7 T1, J8 S1, J9 S2, U1 IP2312U_VSET, U2 XB5606AJ

Commit message: Update PCB
Parts:
- moved C5 37.2 mm to (171.9, 124.0), turned to 180 degrees
- moved R8 35.3 mm to (215.0, 121.0), turned to 90 degrees
- moved R3 35.2 mm to (211.0, 113.2), turned to 90 degrees
- moved R7 34.8 mm to (212.5, 121.0), turned to 90 degrees
- moved R6 34.7 mm to (210.0, 121.0), turned to 90 degrees
- moved R5 34.7 mm to (207.0, 121.0), turned to -90 degrees
- moved R10 34.2 mm to (182.0, 124.2), turned to -90 degrees
- moved R17 33.9 mm to (173.0, 120.0), turned to -90 degrees
- moved R15 32.2 mm to (201.0, 119.8), turned to 90 degrees
- moved J8 31.1 mm to (210.0, 124.3), turned to -90 degrees
- moved J3 30.9 mm to (204.0, 124.3), turned to -90 degrees
- moved R11 30.7 mm to (189.0, 124.2), turned to -90 degrees
- moved R9 30.6 mm to (208.0, 113.2), turned to 90 degrees
- moved J1 30.2 mm to (212.0, 117.0)
- moved R1 29.6 mm to (181.5, 103.0)
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